File: ShroomShed_MKII_PCB/_autosave-ShroomShed_MKII_PCB.kicad_sch (KiCad schematic)
At the start: 68 parts, among them J1 SWD 14 pin header, J2 TYPE-C-31-M-12, J3 Fan, J4 AUX_SPI, J5 SD_SPI, J6 DHT_I2C, J7 Display_Touch_SPI, J8 Front_Panel, J9 Transducer Driver, Q1 T2N7002AK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

Commit message: added solidworks files
Parts:
- renumbered D6 to D3, D3 to D4, R21 to R13, R13 to R14, R14 to R15, R15 to R16
