File: ShroomShed_MKII_PCB/Display_Adapter/Display_Adapter.kicad_pcb (KiCad board)
At the start: 2 copper layers, 16 x 39 mm, 2 parts, among them J1 Display_Touch_SPI, J7 Display_Touch_SPI

Commit message: added solidworks files
Parts:
- J7: footprint DOWNLOAD_Connectors:CONN_532610001-SD_14_MOL -> DOWNLOAD_Connectors:MOLEX_530481410
- moved J7 8.64 mm to (151.1, 93.1), turned to 90 degrees
Connections:
- J7 pad 10: TOUCH_MISO -> TOUCH_SCK
- J7 pad 11: TOUCH_MOSI -> TOUCH_MISO
- J7 pad 12: TOUCH_IRQ -> TOUCH_MOSI
- J7 pad 13: DISPLAY_LED -> TOUCH_IRQ
- J7 pad 8: TOUCH_NSS -> DISPLAY_LED
- J7 pad 9: TOUCH_SCK -> TOUCH_NSS
Routing:
- net GND: track 6.91 -> 0.00 mm, vias 2 -> 0
- net DISPLAY_LED: track 13.0 -> 7.21 mm
- net DISPLAY_MOSI: track 11.4 -> 8.03 mm, vias 1 -> 0
- net TOUCH_MISO: track 18.3 -> 16.2 mm, vias 1 -> 0
- net TOUCH_IRQ: track 13.7 -> 12.4 mm
- net DISPLAY_RST: track 17.9 -> 19.2 mm
- net TOUCH_SCK: track 8.77 -> 7.85 mm
- net TOUCH_MOSI: track 9.84 -> 9.32 mm
- net TOUCH_NSS: track 11.7 -> 11.4 mm, vias 2 -> 0
