File: ShroomShed_MKII_PCB/ERM_PCB/ERM_PCB.kicad_pcb (KiCad board)
At the start: 2 copper layers, 18 x 60 mm, 16 parts, among them J1 Fan, J2 Humidifier, J3 Conn_01x04, Q1 BSS123, Q2 BSS123

Commit message: got the display working thank fuck
Parts:
- J3: footprint DOWNLOAD_Connectors:CONN_532610001-SD_04_MOL -> Connector_JST:JST_XH_S4B-XH-A-1_1x04_P2.50mm_Horizontal
- moved D1 19.6 mm to (191.9, 68.5), turned to 0 degrees
- moved R5 17.5 mm to (188.7, 68.5), turned to 0 degrees
- moved J3 6.10 mm to (191.0, 80.5), turned to 90 degrees
- moved C2 3.94 mm to (195.8, 86.5)
- moved J2 0.86 mm to (191.5, 120.2)
Routing:
- net +12V: track 0.00 -> 12.7 mm
- net HUMIDIFIER_PWM: track 19.3 -> 16.7 mm
- net GND: track 27.3 -> 25.7 mm, vias 2 -> 1
- net FAN_PWM: track 3.89 -> 4.61 mm
Other:
- board text added: "ERM V2.1"
- board text removed: "ERM V1"
